File: Shield.brd (EAGLE design)
At the start: 99.1 x 68.6 mm, 71 parts

Commit message: First completed routing
Parts:
- removed AREFJUMPER: 2PJN, LEMS:2PH
- added U$4: 2PHN, LEMS:2PH
Connections:
- net 4.5V: now also U$4.1, U$4.2; no longer AREFJUMPER.1
- net AREF: no longer AREFJUMPER.2
- net D38: now also 4.7K.1, DALLASTERM.2
- net D39: no longer 4.7K.1, DALLASTERM.2
Routing:
- net D38: track 0.00 -> 89.3 mm, vias 0 -> 2
- net D39: track 36.4 -> 0.00 mm, vias 1 -> 0
- net 4.5V: track 75.2 -> 83.7 mm
- net GND: track 481.4 -> 482.6 mm
Changed lines of the file:
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@@
 <element name="10UF" library="LEMS" package="E2,5-5" value="CES" x="48.006" y="22.86" rot="R270"/>
 <element name="10UF-LOWESR" library="LEMS" package="E2,5-5" value="CES" x="60.452" y="20.32" rot="R270"/>
-<element name="AREFJUMPER" library="LEMS" package="2PH" value="2PJN" x="74.93" y="34.29"/>
 <element name="U$12" library="LEMS" package="DIL16" value="ADS7841P" x="80.01" y="20.32"/>
 <element name="0.1UF-3" library="LEMS" package="C025-025X050" value="CCL" x="66.04" y="25.146" rot="MR180"/>
@@
 <element name="PWRSWTCH" library="LEMS" package="SWITCH-SPDT" value="SWITCHSPDTN" x="9.652" y="17.78" rot="R180"/>
 <element name="PWRTERM" library="LEMS" package="SCREWTERMINAL-3.5MM-2_LOCK" value="2PHS" x="5.08" y="8.382" rot="R270"/>
+<element name="U$4" library="LEMS" package="2PH" value="2PHN" x="58.166" y="24.384" rot="R180"/>
 </elements>
 <signals>
@@
 <wire x1="49.53" y1="21.59" x2="52.07" y2="24.13" width="0.3048" layer="1"/>
 <wire x1="52.07" y1="24.13" x2="53.34" y2="24.13" width="0.3048" layer="1"/>
-<wire x1="53.34" y1="24.13" x2="55.372" y2="24.13" width="0.3048" layer="1"/>
-<wire x1="55.372" y1="24.13" x2="60.452" y2="19.05" width="0.3048" layer="1"/>
 <contactref element="10UF-2" pad="-"/>
 <wire x1="86.36" y1="24.13" x2="83.82" y2="24.13" width="0.3048" layer="1"/>
@@
 <wire x1="10.16" y1="26.67" x2="42.672" y2="26.67" width="0.3048" layer="16"/>
 <wire x1="42.672" y1="26.67" x2="46.482" y2="30.48" width="0.3048" layer="16"/>
+<wire x1="53.34" y1="24.13" x2="54.61" y2="24.13" width="0.3048" layer="16"/>
+<wire x1="54.61" y1="24.13" x2="55.118" y2="23.622" width="0.3048" layer="16"/>
+<wire x1="55.118" y1="23.622" x2="55.118" y2="21.59" width="0.3048" layer="16"/>
+<wire x1="55.118" y1="21.59" x2="55.88" y2="20.828" width="0.3048" layer="16"/>
+<wire x1="55.88" y1="20.828" x2="58.674" y2="20.828" width="0.3048" layer="16"/>
+<wire x1="58.674" y1="20.828" x2="60.452" y2="19.05" width="0.3048" layer="16"/>
 <wire x1="8.89" y1="53.34" x2="6.31" y2="53.34" width="0" layer="19" extent="1-16"/>
 <wire x1="43.053" y1="11.303" x2="42.926" y2="11.303" width="0" layer="19" extent="16-16"/>
@@
 <contactref element="SDLVLS" pad="2"/>
 <contactref element="8-13" pad="5"/>
-<wire x1="34.29" y1="52.07" x2="36.83" y2="54.61" width="0.3048" layer="1"/>
-<wire x1="36.83" y1="54.61" x2="36.83" y2="55.88" width="0.3048" layer="1"/>
 <wire x1="34.29" y1="57.15" x2="30.48" y2="57.15" width="0.3048" layer="16"/>
 <wire x1="30.48" y1="57.15" x2="28.956" y2="58.42" width="0.3048" layer="16"/>
 <wire x1="28.956" y1="58.42" x2="28.956" y2="59.817" width="0.3048" layer="16"/>
 <via x="34.29" y="57.15" extent="1-16" drill="0.6"/>
-<wire x1="34.29" y1="57.15" x2="36.83" y2="55.88" width="0.3048" layer="1"/>
+<wire x1="34.29" y1="52.07" x2="36.322" y2="54.102" width="0.3048" layer="1"/>
+<wire x1="36.322" y1="54.102" x2="36.322" y2="56.134" width="0.3048" layer="1"/>
+<wire x1="36.322" y1="56.134" x2="35.306" y2="57.15" width="0.3048" layer="1"/>
+<wire x1="35.306" y1="57.15" x2="34.29" y2="57.15" width="0.3048" layer="1"/>
 </signal>
 <signal name="SD_SCKIN">
@@
 <signal name="AREF">
 <contactref element="8-13" pad="3"/>
-<contactref element="AREFJUMPER" pad="2"/>
-<wire x1="23.876" y1="59.817" x2="76.3778" y2="34.29" width="0" layer="19" extent="1-1"/>
 </signal>
 <signal name="D7">
@@
 <contactref element="0-7" pad="5"/>
 <contactref element="TN9TERM" pad="2"/>
-<wire x1="55.88" y1="59.817" x2="52.705" y2="62.992" width="0.3048" layer="1"/>
-<wire x1="52.705" y1="62.992" x2="50.038" y2="62.992" width="0.3048" layer="1"/>
-<wire x1="50.038" y1="62.992" x2="48.57" y2="64.46" width="0.3048" layer="1"/>
-<wire x1="48.57" y1="64.46" x2="48.57" y2="64.77" width="0.3048" layer="1"/>
+<wire x1="55.88" y1="59.817" x2="53.467" y2="62.23" width="0.3048" layer="1"/>
+<wire x1="53.467" y1="62.23" x2="52.07" y2="62.23" width="0.3048" layer="1"/>
+<wire x1="52.07" y1="62.23" x2="49.53" y2="64.77" width="0.3048" layer="1"/>
+<wire x1="49.53" y1="64.77" x2="48.57" y2="64.77" width="0.3048" layer="1"/>
 </signal>
 <signal name="TN9_DATA">
@@
 <signal name="D39">
 <contactref element="39-53" pad="1"/>
-<contactref element="DALLASTERM" pad="2"/>
-<contactref element="4.7K" pad="1"/>
-<wire x1="68.524" y1="6.35" x2="68.524" y2="6.66" width="0.3048" layer="1"/>
-<wire x1="68.524" y1="6.66" x2="65.532" y2="9.652" width="0.3048" layer="1"/>
-<wire x1="65.532" y1="9.652" x2="50.038" y2="9.652" width="0.3048" layer="1"/>
-<wire x1="50.038" y1="9.652" x2="49.022" y2="10.668" width="0.3048" layer="1"/>
-<wire x1="49.022" y1="10.668" x2="49.022" y2="12.192" width="0.3048" layer="1"/>
-<wire x1="49.022" y1="12.192" x2="50.8" y2="13.97" width="0.3048" layer="1"/>
-<wire x1="50.8" y1="13.97" x2="57.658" y2="13.97" width="0.3048" layer="1"/>
-<via x="58.166" y="14.478" extent="1-16" drill="0.6"/>
-<wire x1="58.166" y1="14.478" x2="59.436" y2="15.748" width="0.3048" layer="16"/>
-<wire x1="59.436" y1="15.748" x2="60.96" y2="15.748" width="0.3048" layer="16"/>
-<wire x1="57.658" y1="13.97" x2="58.166" y2="14.478" width="0.3048" layer="1"/>
-<wire x1="68.524" y1="6.66" x2="96.647" y2="36.83" width="0" layer="19" extent="1-1"/>
 </signal>
 <signal name="D41">
@@
 <signal name="D38">
 <contactref element="38-52" pad="1"/>
+<contactref element="DALLASTERM" pad="2"/>
+<contactref element="4.7K" pad="1"/>
+<wire x1="68.524" y1="6.35" x2="68.524" y2="6.66" width="0.3048" layer="1"/>
+<wire x1="68.524" y1="6.66" x2="65.532" y2="9.652" width="0.3048" layer="1"/>
+<wire x1="65.532" y1="9.652" x2="50.038" y2="9.652" width="0.3048" layer="1"/>
+<wire x1="50.038" y1="9.652" x2="49.022" y2="10.668" width="0.3048" layer="1"/>
+<wire x1="49.022" y1="10.668" x2="49.022" y2="12.192" width="0.3048" layer="1"/>
+<wire x1="49.022" y1="12.192" x2="50.8" y2="13.97" width="0.3048" layer="1"/>
+<wire x1="50.8" y1="13.97" x2="57.658" y2="13.97" width="0.3048" layer="1"/>
+<via x="58.166" y="14.478" extent="1-16" drill="0.6"/>
+<wire x1="58.166" y1="14.478" x2="59.436" y2="15.748" width="0.3048" layer="16"/>
+<wire x1="59.436" y1="15.748" x2="60.96" y2="15.748" width="0.3048" layer="16"/>
+<wire x1="57.658" y1="13.97" x2="58.166" y2="14.478" width="0.3048" layer="1"/>
+<wire x1="60.96" y1="15.748" x2="60.96" y2="16.764" width="0.3048" layer="16"/>
+<wire x1="60.96" y1="16.764" x2="61.722" y2="17.526" width="0.3048" layer="16"/>
+<wire x1="61.722" y1="17.526" x2="62.738" y2="17.526" width="0.3048" layer="16"/>
+<wire x1="62.738" y1="17.526" x2="63.246" y2="18.034" width="0.3048" layer="16"/>
+<wire x1="63.246" y1="18.034" x2="63.246" y2="23.114" width="0.3048" layer="16"/>
+<wire x1="63.246" y1="23.114" x2="62.23" y2="24.13" width="0.3048" layer="16"/>
+<wire x1="62.23" y1="24.13" x2="62.23" y2="26.924" width="0.3048" layer="1"/>
+<wire x1="62.23" y1="26.924" x2="62.484" y2="27.178" width="0.3048" layer="1"/>
+<wire x1="62.484" y1="27.178" x2="90.932" y2="27.178" width="0.3048" layer="1"/>
+<wire x1="90.932" y1="27.178" x2="91.694" y2="27.94" width="0.3048" layer="1"/>
+<wire x1="91.694" y1="27.94" x2="91.694" y2="34.417" width="0.3048" layer="1"/>
+<wire x1="91.694" y1="34.417" x2="94.107" y2="36.83" width="0.3048" layer="1"/>
+<via x="62.23" y="24.13" extent="1-16" drill="0.6"/>
 </signal>
 <signal name="D40">
@@
 <contactref element="4.5VTERM" pad="1"/>
 <contactref element="4.5VTERM" pad="2"/>
-<contactref element="AREFJUMPER" pad="1"/>
 <contactref element="U$12" pad="8"/>
 <wire x1="88.9" y1="16.51" x2="86.36" y2="13.97" width="0.3048" layer="1"/>
@@
 <wire x1="57.658" y1="17.145" x2="55.9562" y2="17.145" width="0.3048" layer="1"/>
 <wire x1="60.452" y1="21.59" x2="58.42" y2="19.558" width="0.3048" layer="1"/>
-<wire x1="58.42" y1="19.558" x2="58.42" y2="16.764" width="0.3048" layer="1"/>
+<wire x1="58.42" y1="19.558" x2="58.42" y2="19.05" width="0.3048" layer="1"/>
+<wire x1="58.42" y1="19.05" x2="58.42" y2="16.764" width="0.3048" layer="1"/>
 <wire x1="57.2262" y1="6.35" x2="61.0818" y2="6.35" width="0.3048" layer="1"/>
 <wire x1="61.0818" y1="6.35" x2="61.0818" y2="7.4982" width="0.3048" layer="1"/>
@@
 <wire x1="56.896" y1="14.732" x2="57.658" y2="15.494" width="0.3048" layer="1"/>
 <wire x1="57.658" y1="15.494" x2="57.658" y2="17.145" width="0.3048" layer="1"/>
-<wire x1="60.452" y1="21.59" x2="73.4822" y2="34.29" width="0" layer="19" extent="1-1"/>
+<contactref element="U$4" pad="2"/>
+<contactref element="U$4" pad="1"/>
+<wire x1="56.7182" y1="24.384" x2="59.6138" y2="24.384" width="0.3048" layer="1"/>
+<wire x1="56.7182" y1="24.384" x2="56.7182" y2="22.0218" width="0.3048" layer="1"/>
+<wire x1="56.7182" y1="22.0218" x2="58.42" y2="20.32" width="0.3048" layer="1"/>
+<wire x1="58.42" y1="20.32" x2="58.42" y2="19.558" width="0.3048" layer="1"/>
 </signal>
 <signal name="CH0">
