File: Shield.brd (EAGLE design)
At the start: 99.1 x 71.1 mm, 80 parts

Commit message: Added middle screw terminals
Parts:
- added U$16: 2PHS, LEMS:SCREWTERMINAL-3.5MM-2_LOCK
- added U$7: 3PHS, LEMS:SCREWTERMINAL-3.5MM-3_LOCK.007S
Connections:
- removed net D5: 0-7.3
- new net D2: 0-7.6, U$7.1
- net D6: now also U$7.2
- net D7: now also U$7.3
- net GND: now also U$16.1, U$16.2
- net TN9_ACT: now also TN9TERM.2; no longer TN9TERM.3
- net TN9_CLK: now also TN9TERM.1; no longer TN9TERM.2
- net TN9_DATA: now also 0-7.3, TN9TERM.3; no longer 0-7.6, TN9TERM.1
Routing:
- net GND: track 460.9 -> 494.1 mm
- net D6: track 0.00 -> 14.8 mm
- net D7: track 0.00 -> 14.6 mm
- net D2: track 0.00 -> 13.2 mm
- net TN9_ACT: track 9.84 -> 6.87 mm
- net TN9_CLK: track 8.60 -> 6.14 mm
Other:
- board text added: "3.3"
- board text added: "MechE"
- board text added: "SCL"
- board text added: "SDA"
- board text added: "SOLR CELL"
- board text removed: "SCL3"
- board text removed: "SCL5"
- board text removed: "SDA3"
- board text removed: "SDA5"
- board text removed: "SOLAR"

Commit message: Minor Spacing Changes
Parts:
- moved U$16 2.54 mm to (64.8, 44.5)
- moved U$7 2.54 mm to (57.1, 44.5)
- renumbered 1 to 0.5, 6.8UF-T to 10UF-T
Routing:
- net D6: track 14.8 -> 18.1 mm
- net GND: track 494.1 -> 491.3 mm
- net D7: track 14.6 -> 17.1 mm
- net D2: track 13.2 -> 15.7 mm

Commit message: Ready for Quantity Manufacturing
Parts:
- 4.7K: value RESISTORT -> RN; device LEMS:0207/7 -> LEMS:0207/10
- moved BMP085TERM 1.27 mm to (83.6, 39.9)
Routing:
- net GND: track 491.3 -> 489.5 mm
- net 3.3V: track 129.9 -> 131.5 mm
- net 5V: track 288.8 -> 288.1 mm
Other:
- board text removed: "38"
Changed lines of the file:
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@@
 <text x="77.978" y="57.15" size="1.016" layer="21" rot="SR0">18</text>
 <text x="80.518" y="57.15" size="1.016" layer="21" rot="SR0">19</text>
-<text x="90.678" y="36.322" size="1.016" layer="21">38</text>
 <text x="90.678" y="33.782" size="1.016" layer="21">40</text>
 <text x="90.678" y="31.242" size="1.016" layer="21">42</text>
@@
 <text x="83.058" y="57.15" size="1.016" layer="21">20</text>
 <text x="85.598" y="57.15" size="1.016" layer="21">21</text>
-<text x="74.168" y="39.624" size="1.016" layer="21">VCC</text>
+<text x="72.898" y="39.624" size="1.016" layer="21">VCC</text>
 <text x="90.678" y="57.15" size="1.016" layer="21">22</text>
 <text x="68.072" y="12.954" size="1.016" layer="21">A7</text>
@@
 <vertex x="46.99" y="30.48"/>
 <vertex x="46.99" y="25.4"/>
+</polygon>
+<polygon width="0.3048" layer="21">
+<vertex x="53.34" y="30.48"/>
+<vertex x="54.61" y="30.48"/>
+<vertex x="54.61" y="31.75"/>
+<vertex x="55.88" y="31.75"/>
+<vertex x="55.88" y="33.02"/>
+<vertex x="53.34" y="33.02"/>
 </polygon>
 </plain>
@@
 <element name="OPA2TERM" library="LEMS" package="3PH" value="3PHN" x="63.5" y="32.766" rot="R180"/>
 <element name="DALLASTERM" library="LEMS" package="SCREWTERMINAL-3.5MM-3_LOCK.007S" value="3PHS" x="65.024" y="6.35"/>
-<element name="4.7K" library="LEMS" package="0207/7" value="RESISTORT" x="85.09" y="36.83" rot="MR0"/>
+<element name="4.7K" library="LEMS" package="0207/10" value="RN" x="85.09" y="36.83" rot="MR0"/>
 <element name="4.5VTERM" library="LEMS" package="SCREWTERMINAL-3.5MM-2_LOCK" value="2PHS" x="57.404" y="6.35"/>
 <element name="ADCTERM" library="LEMS" package="SCREWTERMINAL-3.5MM-3_LOCK.007S" value="3PHS" x="76.708" y="6.35"/>
@@
 <element name="GNDTERM" library="LEMS" package="SCREWTERMINAL-3.5MM-3_LOCK.007S" value="3PHS" x="27.432" y="6.35"/>
 <element name="3.3VTERM" library="LEMS" package="SCREWTERMINAL-3.5MM-3_LOCK.007S" value="3PHS" x="15.748" y="6.35"/>
-<element name="BMP085TERM" library="LEMS" package="6PH" value="6PHN" x="84.836" y="39.878" rot="R180"/>
+<element name="BMP085TERM" library="LEMS" package="6PH" value="6PHN" x="83.566" y="39.878" rot="R180"/>
 <element name="OPAMPEXTRA1" library="LEMS" package="3PH" value="3PHN" x="63.5" y="38.354" rot="R180"/>
 <element name="OPAMPEXTRA2" library="LEMS" package="3PH" value="3PHN" x="63.5" y="35.56" rot="R180"/>
@@
 <wire x1="47.879" y1="16.51" x2="43.18" y2="11.811" width="0.8128" layer="1"/>
 <wire x1="43.18" y1="11.811" x2="43.18" y2="11.557" width="0.8128" layer="1"/>
-<wire x1="80.772" y1="38.1" x2="73.66" y2="38.1" width="0.3048" layer="16"/>
-<wire x1="73.66" y1="38.1" x2="73.406" y2="37.846" width="0.3048" layer="16"/>
-<wire x1="73.406" y1="37.846" x2="73.406" y2="35.56" width="0.3048" layer="16"/>
+<wire x1="73.406" y1="38.1" x2="73.406" y2="35.56" width="0.3048" layer="16"/>
 <wire x1="27.2542" y1="6.35" x2="30.932" y2="6.35" width="0.8128" layer="16"/>
 <wire x1="34.544" y1="6.2842" x2="30.9978" y2="6.2842" width="0.8128" layer="16"/>
 <wire x1="30.9978" y1="6.2842" x2="30.932" y2="6.35" width="0.8128" layer="16"/>
-<wire x1="78.486" y1="47.752" x2="81.026" y2="45.212" width="0.3048" layer="1"/>
-<wire x1="81.026" y1="45.212" x2="81.026" y2="39.878" width="0.3048" layer="1"/>
-<wire x1="81.026" y1="39.878" x2="81.026" y2="38.354" width="0.3048" layer="16"/>
-<wire x1="81.026" y1="38.354" x2="80.772" y2="38.1" width="0.3048" layer="16"/>
 <contactref element="U$16" pad="1"/>
 <contactref element="U$16" pad="2"/>
@@
 <wire x1="60.96" y1="41.402" x2="60.96" y2="44.3178" width="0.3048" layer="1"/>
 <wire x1="60.96" y1="44.3178" x2="61.0922" y2="44.45" width="0.3048" layer="1"/>
-<wire x1="73.406" y1="37.846" x2="64.9478" y2="44.45" width="0" layer="19" extent="16-16"/>
+<wire x1="73.406" y1="38.1" x2="73.66" y2="38.354" width="0.3048" layer="16"/>
+<wire x1="73.66" y1="38.354" x2="79.502" y2="38.354" width="0.3048" layer="16"/>
+<wire x1="79.502" y1="38.354" x2="79.756" y2="38.608" width="0.3048" layer="16"/>
+<wire x1="79.756" y1="38.608" x2="79.756" y2="39.878" width="0.3048" layer="16"/>
+<wire x1="79.756" y1="39.878" x2="79.756" y2="42.418" width="0.3048" layer="1"/>
+<wire x1="79.756" y1="42.418" x2="78.486" y2="43.688" width="0.3048" layer="1"/>
+<wire x1="78.486" y1="43.688" x2="78.486" y2="47.752" width="0.3048" layer="1"/>
+<wire x1="73.406" y1="38.1" x2="64.9478" y2="44.45" width="0" layer="19" extent="16-16"/>
 </signal>
 <signal name="MOSI_SOFT">
@@
 <wire x1="56.896" y1="32.258" x2="56.896" y2="39.116" width="0.3048" layer="16"/>
 <wire x1="56.896" y1="39.116" x2="57.912" y2="40.132" width="0.3048" layer="16"/>
-<wire x1="78.486" y1="40.132" x2="57.912" y2="40.132" width="0.3048" layer="16"/>
-<wire x1="83.058" y1="43.18" x2="81.534" y2="43.18" width="0.3048" layer="16"/>
-<wire x1="81.534" y1="43.18" x2="78.486" y2="40.132" width="0.3048" layer="16"/>
+<wire x1="83.058" y1="43.18" x2="82.296" y2="43.18" width="0.3048" layer="16"/>
+<wire x1="82.296" y1="43.18" x2="81.534" y2="43.18" width="0.3048" layer="16"/>
+<wire x1="57.912" y1="40.132" x2="77.216" y2="40.132" width="0.3048" layer="16"/>
+<wire x1="77.216" y1="40.132" x2="77.216" y2="42.926" width="0.3048" layer="16"/>
+<wire x1="77.216" y1="42.926" x2="77.47" y2="43.18" width="0.3048" layer="16"/>
+<wire x1="77.47" y1="43.18" x2="81.534" y2="43.18" width="0.3048" layer="16"/>
 </signal>
 <signal name="5V">
@@
 <wire x1="71.374" y1="51.562" x2="70.866" y2="52.07" width="0.254" layer="1"/>
 <wire x1="70.866" y1="52.07" x2="70.866" y2="55.372" width="0.254" layer="1"/>
-<wire x1="81.28" y1="36.83" x2="81.28" y2="33.528" width="0.254" layer="1"/>
 <wire x1="81.28" y1="33.528" x2="83.312" y2="33.528" width="0.254" layer="1"/>
 <wire x1="83.312" y1="33.528" x2="83.566" y2="33.274" width="0.254" layer="1"/>
@@
 <wire x1="65.024" y1="39.116" x2="65.024" y2="37.338" width="0.3048" layer="1"/>
 <wire x1="65.024" y1="37.338" x2="65.278" y2="37.084" width="0.3048" layer="1"/>
-<wire x1="65.278" y1="37.084" x2="74.93" y2="37.084" width="0.3048" layer="1"/>
-<wire x1="74.93" y1="37.084" x2="81.026" y2="37.084" width="0.3048" layer="1"/>
-<wire x1="81.026" y1="37.084" x2="81.28" y2="36.83" width="0.3048" layer="1"/>
+<wire x1="65.278" y1="37.084" x2="74.422" y2="37.084" width="0.3048" layer="1"/>
+<wire x1="74.422" y1="37.084" x2="74.93" y2="37.084" width="0.3048" layer="1"/>
 <wire x1="75.946" y1="35.56" x2="75.946" y2="36.068" width="0.3048" layer="1"/>
 <wire x1="75.946" y1="36.068" x2="74.93" y2="37.084" width="0.3048" layer="1"/>
-<wire x1="81.026" y1="37.084" x2="81.788" y2="48.26" width="0" layer="19" extent="1-1"/>
+<wire x1="81.28" y1="33.528" x2="81.28" y2="35.56" width="0.254" layer="1"/>
+<wire x1="81.28" y1="35.56" x2="80.01" y2="36.83" width="0.254" layer="1"/>
+<wire x1="80.01" y1="36.83" x2="77.47" y2="36.83" width="0.3048" layer="1"/>
+<wire x1="77.47" y1="36.83" x2="77.216" y2="37.084" width="0.3048" layer="1"/>
+<wire x1="77.216" y1="37.084" x2="74.93" y2="37.084" width="0.3048" layer="1"/>
+<wire x1="80.01" y1="36.83" x2="81.788" y2="48.26" width="0" layer="19" extent="1-1"/>
 </signal>
 <signal name="I2C-2">
@@
 <contactref element="DALLASTERM" pad="2"/>
 <contactref element="4.7K" pad="1"/>
-<wire x1="88.9" y1="36.83" x2="94.107" y2="36.83" width="0.254" layer="1"/>
 <wire x1="68.524" y1="6.35" x2="68.524" y2="7.056" width="0.254" layer="1"/>
 <wire x1="68.524" y1="7.056" x2="72.136" y2="10.668" width="0.254" layer="1"/>
@@
 <wire x1="72.644" y1="12.954" x2="84.582" y2="12.954" width="0.254" layer="1"/>
 <wire x1="84.582" y1="12.954" x2="85.09" y2="13.462" width="0.254" layer="1"/>
+<wire x1="90.17" y1="36.83" x2="94.107" y2="36.83" width="0.254" layer="1"/>
 <wire x1="85.09" y1="13.462" x2="85.09" y2="36.322" width="0.254" layer="1"/>
 <wire x1="85.09" y1="36.322" x2="85.598" y2="36.83" width="0.254" layer="1"/>
-<wire x1="85.598" y1="36.83" x2="88.9" y2="36.83" width="0.254" layer="1"/>
+<wire x1="85.598" y1="36.83" x2="90.17" y2="36.83" width="0.254" layer="1"/>
 </signal>
 <signal name="D40">
@@
 <wire x1="90.932" y1="61.976" x2="90.932" y2="55.245" width="0.254" layer="16"/>
 <wire x1="90.932" y1="55.245" x2="91.059" y2="55.118" width="0.254" layer="16"/>
-<wire x1="90.678" y1="43.18" x2="91.186" y2="42.672" width="0.254" layer="1"/>
-<wire x1="91.186" y1="42.672" x2="91.186" y2="39.878" width="0.254" layer="1"/>
+<wire x1="89.916" y1="39.878" x2="89.916" y2="42.418" width="0.254" layer="1"/>
+<wire x1="89.916" y1="42.418" x2="90.678" y2="43.18" width="0.254" layer="1"/>
 </signal>
 <signal name="3.3V_SCL">
@@
 <wire x1="90.678" y1="45.72" x2="90.678" y2="49.911" width="0.254" layer="1"/>
 <wire x1="90.678" y1="49.911" x2="91.059" y2="50.292" width="0.254" layer="1"/>
-<wire x1="90.678" y1="45.72" x2="89.154" y2="45.72" width="0.254" layer="1"/>
-<wire x1="89.154" y1="45.72" x2="88.646" y2="45.212" width="0.254" layer="1"/>
-<wire x1="88.646" y1="45.212" x2="88.646" y2="40.132" width="0.254" layer="1"/>
+<wire x1="87.376" y1="40.132" x2="87.376" y2="42.418" width="0.254" layer="1"/>
+<wire x1="87.376" y1="42.418" x2="90.678" y2="45.72" width="0.254" layer="1"/>
 </signal>
 <signal name="REDLED">
