File: Shield.sch (EAGLE design)
At the start: 71 parts

Commit message: Improved Routing
Connections:
- net CH1: now also ADCTERM.1; no longer ADCTERM.3
- net CH3: now also ADCTERM.3; no longer ADCTERM.1
- net MISO: now also SPITERM.1; no longer SPITERM.3
- net MOSI: now also SPITERM.3; no longer SPITERM.2
- net SCK: now also SPITERM.2; no longer SPITERM.1

Commit message: Continued routing
Connections:
- net 5V: now also 10UF-2.1; no longer 10UF-2.2
- net GND: now also 10UF-2.2; no longer 10UF-2.1
Other:
- moved on the sheet: 10UF-2
Changed lines of the file:
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@@
 <instance part="U$13" gate="G$1" x="137.16" y="88.9"/>
 <instance part="0.1UF-3" gate="G$1" x="139.7" y="104.14"/>
-<instance part="10UF-2" gate="G$1" x="149.86" y="104.14"/>
+<instance part="10UF-2" gate="G$1" x="149.86" y="104.14" rot="R180"/>
 <instance part="GND15" gate="1" x="144.78" y="116.84" rot="R180"/>
 <instance part="U$14" gate="TLV2372-1" x="190.5" y="127"/>
@@
 <pinref part="0.1UF-3" gate="G$1" pin="1"/>
 <wire x1="139.7" y1="106.68" x2="139.7" y2="114.3" width="0.1524" layer="91"/>
-<pinref part="10UF-2" gate="G$1" pin="1"/>
 <wire x1="139.7" y1="114.3" x2="144.78" y2="114.3" width="0.1524" layer="91"/>
 <wire x1="144.78" y1="114.3" x2="149.86" y2="114.3" width="0.1524" layer="91"/>
-<wire x1="149.86" y1="114.3" x2="149.86" y2="106.68" width="0.1524" layer="91"/>
 <pinref part="GND15" gate="1" pin="GND"/>
 <junction x="144.78" y="114.3"/>
+<pinref part="10UF-2" gate="G$1" pin="2"/>
+<wire x1="149.86" y1="109.22" x2="149.86" y2="114.3" width="0.1524" layer="91"/>
 </segment>
 <segment>
@@
 <segment>
 <pinref part="U$12" gate="ADS7841" pin="VCC"/>
-<wire x1="152.4" y1="88.9" x2="149.86" y2="88.9" width="0.1524" layer="91"/>
 <pinref part="U$13" gate="G$1" pin="5V"/>
 <pinref part="0.1UF-3" gate="G$1" pin="2"/>
+<wire x1="152.4" y1="88.9" x2="149.86" y2="88.9" width="0.1524" layer="91"/>
 <wire x1="149.86" y1="88.9" x2="144.78" y2="88.9" width="0.1524" layer="91"/>
 <wire x1="144.78" y1="88.9" x2="139.7" y2="88.9" width="0.1524" layer="91"/>
@@
 <wire x1="139.7" y1="88.9" x2="139.7" y2="99.06" width="0.1524" layer="91"/>
 <junction x="139.7" y="88.9"/>
-<pinref part="10UF-2" gate="G$1" pin="2"/>
-<wire x1="149.86" y1="88.9" x2="149.86" y2="99.06" width="0.1524" layer="91"/>
-<junction x="149.86" y="88.9"/>
 <pinref part="U$12" gate="ADS7841" pin="/SHDN"/>
 <wire x1="152.4" y1="58.42" x2="144.78" y2="58.42" width="0.1524" layer="91"/>
 <wire x1="144.78" y1="58.42" x2="144.78" y2="88.9" width="0.1524" layer="91"/>
 <junction x="144.78" y="88.9"/>
-</segment>
-<segment>
+<pinref part="10UF-2" gate="G$1" pin="1"/>
+<wire x1="149.86" y1="101.6" x2="149.86" y2="88.9" width="0.1524" layer="91"/>
+<junction x="149.86" y="88.9"/>
+</segment>
+<segment>

Commit message: Almost complete routing
Connections:
- net GND: now also OPA1TERM.2; no longer OPA1TERM.1
- net LIOP-: now also OPA1TERM.1; no longer OPA1TERM.2
Changed lines of the file:
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@@
 </segment>
 <segment>
-<pinref part="OPA1TERM" gate="G$1" pin="1"/>
-<wire x1="165.1" y1="127" x2="167.64" y2="127" width="0.1524" layer="91"/>
-<wire x1="167.64" y1="127" x2="167.64" y2="124.46" width="0.1524" layer="91"/>
 <pinref part="U$14" gate="TLV2372-1" pin="+IN"/>
 <wire x1="167.64" y1="124.46" x2="175.26" y2="124.46" width="0.1524" layer="91"/>
@@
 <wire x1="175.26" y1="124.46" x2="185.42" y2="124.46" width="0.1524" layer="91"/>
 <junction x="175.26" y="124.46"/>
+<wire x1="167.64" y1="124.46" x2="167.64" y2="129.54" width="0.1524" layer="91"/>
+<pinref part="OPA1TERM" gate="G$1" pin="2"/>
+<wire x1="167.64" y1="129.54" x2="165.1" y2="129.54" width="0.1524" layer="91"/>
 </segment>
 <segment>
@@
 <net name="LIOP-" class="0">
 <segment>
-<pinref part="OPA1TERM" gate="G$1" pin="2"/>
 <pinref part="U$14" gate="TLV2372-1" pin="-IN"/>
-<wire x1="165.1" y1="129.54" x2="175.26" y2="129.54" width="0.1524" layer="91"/>
 <wire x1="175.26" y1="129.54" x2="185.42" y2="129.54" width="0.1524" layer="91"/>
 <wire x1="175.26" y1="129.54" x2="175.26" y2="137.16" width="0.1524" layer="91"/>
-<junction x="175.26" y="129.54"/>
 <pinref part="1UF-2" gate="G$1" pin="1"/>
 <wire x1="175.26" y1="137.16" x2="175.26" y2="144.78" width="0.1524" layer="91"/>
@@
 <junction x="175.26" y="137.16"/>
 <label x="170.18" y="144.78" size="1.27" layer="95"/>
-</segment>
-</net>
+<wire x1="175.26" y1="129.54" x2="170.18" y2="129.54" width="0.1524" layer="91"/>
+<wire x1="170.18" y1="129.54" x2="170.18" y2="127" width="0.1524" layer="91"/>
+<junction x="175.26" y="129.54"/>
+<pinref part="OPA1TERM" gate="G$1" pin="1"/>
+<wire x1="170.18" y1="127" x2="165.1" y2="127" width="0.1524" layer="91"/>
+<label x="177.8" y="129.54" size="1.778" layer="95"/>
+</segment>
+</net>

Commit message: First completed routing
Parts:
- removed AREFJUMPER: 2PJN, LEMS:2PJN
- added U$4: 2PHN, LEMS:2PHN
Connections:
- net 4.5V: now also U$4.1, U$4.2; no longer AREFJUMPER.1
- net AREF: no longer AREFJUMPER.2
- net D38: now also 4.7K.1, DALLASTERM.2
- net D39: no longer 4.7K.1, DALLASTERM.2
